File: KiCAD/vael.kicad_pcb (KiCad board)
At the start: 2 copper layers, 61 x 61 mm, 68 parts, among them J1 Micro_SD_Card, J2 USB_C_Receptacle_USB2.0_16P, J3 Conn_01x03, J4 Conn_01x03, J5 Conn_01x03, J6 Conn_01x03, J7 Conn_01x04, Q1 FS8205A, SW1 SW_SPST, SW2 SW_SPDT, U1 ESP32-S3-WROOM-1-N8R8, U2 DW01A, U3 USBLC6-2SC6, U4 TP4056, U5 MT3608, U6 AMS1117-3.3, U7 MPU-6050, U8 BMP18

Commit message: test firmware
Parts:
- removed dialgorithm (x2): dialgorithm, dialgorithm:dialgorithm
